Commit message: Fix camera orientation

File: ca_description/urdf/roomblock.urdf.xacro (robot description, xacro)
@@ -34,5 +34,5 @@
     <link name="laser_link"/>
     <joint name="camera_joint" type="fixed">
-      <origin xyz="${camera_x_offset} 0 ${camera_z_offset}" rpy="0 ${pi/2} 0" />
+      <origin xyz="${camera_x_offset} 0 ${camera_z_offset}" rpy="0 0 0" />
       <parent link="block_link" />
       <child link="raspicam_link" />
