Commit message: Edit Create 2 model with block and fixes

File: ca_description/urdf/create_2.urdf.xacro (robot description, xacro)
@@ -1,8 +1,10 @@
 <?xml version="1.0" ?>
 <robot name="create_2" xmlns:xacro="http://ros.org/wiki/xacro">
-  <xacro:include filename="$(find ca_description)/urdf/create_base.urdf.xacro" />
-  <xacro:include filename="$(find ca_description)/urdf/create_2_gazebo.urdf.xacro" />
+  <xacro:include filename="$(find ca_description)/urdf/create_base.urdf.xacro"/>
+  <xacro:include filename="$(find ca_description)/urdf/roomblock.urdf.xacro"/>
   <xacro:create_base wheel_separation="0.235" base_diameter="0.3485">
     <mesh filename="package://ca_description/meshes/create_2.dae" />
   </xacro:create_base>
+  <!-- Roomblock -->
+  <xacro:roomblock/>
 </robot>

File: ca_description/urdf/create_base.urdf.xacro (robot description, xacro)
@@ -1,5 +1,4 @@
 <?xml version="1.0" ?>
 <robot xmlns:xacro="http://ros.org/wiki/xacro">
-  <xacro:property name="PI" value="3.1415926535897931" />
   <xacro:macro name="create_wheel" params="prefix y_offset wheel_radius wheel_width">
     <link name="${prefix}_wheel_link">
@@ -10,5 +9,5 @@
     </inertial>
     <visual>
-      <origin xyz="0 0 0" rpy="0 ${PI/2} ${PI/2}" />
+      <origin xyz="0 0 0" rpy="0 ${pi/2} ${pi/2}" />
       <geometry>
         <cylinder radius="${wheel_radius}" length="${wheel_width}" />
@@ -16,5 +15,5 @@
     </visual>
     <collision>
-      <origin xyz="0 0 0" rpy="0 ${PI/2} ${PI/2}" />
+      <origin xyz="0 0 0" rpy="0 ${pi/2} ${pi/2}" />
       <geometry>
         <cylinder radius="${wheel_radius}" length="${wheel_width}" />
@@ -111,20 +110,20 @@
     </joint>
     <joint name="base_left_cliff_sensor_joint" type="fixed">
-      <origin xyz="0.07 0.14 0.01" rpy="0 ${PI/2} 0" />
+      <origin xyz="0.07 0.14 0.01" rpy="0 ${pi/2} 0" />
       <parent link="base_link" />
       <child link="left_cliff_sensor_link" />
     </joint>
     <joint name="base_right_cliff_sensor_joint" type="fixed">
-      <origin xyz="0.07 -0.14 0.01" rpy="0 ${PI/2} 0" />
+      <origin xyz="0.07 -0.14 0.01" rpy="0 ${pi/2} 0" />
       <parent link="base_link" />
       <child link="right_cliff_sensor_link" />
     </joint>
     <joint name="base_leftfront_cliff_sensor_joint" type="fixed">
-      <origin xyz="0.15 0.04 0.01" rpy="0 ${PI/2} 0" />
+      <origin xyz="0.15 0.04 0.01" rpy="0 ${pi/2} 0" />
       <parent link="base_link" />
       <child link="leftfront_cliff_sensor_link" />
     </joint>
     <joint name="base_rightfront_cliff_sensor_joint" type="fixed">
-      <origin xyz="0.15 -0.04 0.01" rpy="0 ${PI/2} 0" />
+      <origin xyz="0.15 -0.04 0.01" rpy="0 ${pi/2} 0" />
       <parent link="base_link" />
       <child link="rightfront_cliff_sensor_link" />
@@ -132,30 +131,4 @@
     <xacro:create_wheel prefix="left" y_offset="${wheel_separation / 2}" wheel_radius="${wheel_radius}" wheel_width="${wheel_width}"/>
     <xacro:create_wheel prefix="right" y_offset="${wheel_separation / -2}" wheel_radius="${wheel_radius}" wheel_width="${wheel_width}"/>
-    <!--<link name="rear_wheel_link">
-    <inertial>
-      <origin xyz="0 0 0"/>
-      <mass value="0.001" />
-      <inertia ixx="0.0001" ixy="0.0" ixz="0.0"
-        iyy="0.0001" iyz="0.0" izz="0.0001" />
-    </inertial>
-    <visual>
-      <origin xyz="0 0 0" rpy="0 ${PI/2} ${PI/2}"/>
-      <geometry>
-        <sphere radius="0.015" />
-      </geometry>
-    </visual>
-    <collision>
-      <origin xyz="0 0 0" rpy="0 ${PI/2} ${PI/2}" />
-      <geometry>
-        <sphere radius="0.015" />
-      </geometry>
-    </collision>
-    </link>
-    <joint name="rear_castor_joint" type="fixed">
-      <origin xyz="-0.13 0 0.0" rpy="0 0 0"/>
-      <parent link="base_link"/>
-      <child link="rear_wheel_link"/>
-      <axis xyz="0 1 0"/>
-    </joint>-->
     <link name="front_wheel_link">
     <inertial>
@@ -165,5 +138,5 @@
     </inertial>
     <visual>
-      <origin xyz="0 0 0" rpy="0 ${PI/2} ${PI/2}" />
+      <origin xyz="0 0 0" rpy="0 ${pi/2} ${pi/2}" />
       <geometry>
         <sphere radius="0.018" />
@@ -171,5 +144,5 @@
     </visual>
     <collision>
-      <origin xyz="0 0 0" rpy="0 ${PI/2} ${PI/2}" />
+      <origin xyz="0 0 0" rpy="0 ${pi/2} ${pi/2}" />
       <geometry>
         <sphere radius="0.018" />

File: ca_description/urdf/create_base_gazebo.urdf.xacro (robot description, xacro)
@@ -21,5 +21,5 @@
         <publishWheelJointState>true</publishWheelJointState>
         <legacyMode>true</legacyMode>
-        <odometrySource>1</odometrySource>
+        <odometrySource>world</odometrySource>
         <publishTf>1</publishTf>
       </plugin>

Commit message: Add visualize flag for seeing lasers

File: ca_description/urdf/create_2.urdf.xacro (robot description, xacro)
@@ -3,8 +3,8 @@
   <xacro:include filename="$(find ca_description)/urdf/create_base.urdf.xacro"/>
   <xacro:include filename="$(find ca_description)/urdf/roomblock.urdf.xacro"/>
-  <xacro:create_base wheel_separation="0.235" base_diameter="0.3485">
+  <xacro:create_base wheel_separation="0.235" base_diameter="0.3485" visualize="$(arg visualize)">
     <mesh filename="package://ca_description/meshes/create_2.dae" />
   </xacro:create_base>
   <!-- Roomblock -->
-  <xacro:roomblock/>
+  <xacro:roomblock visualize="$(arg visualize)"/>
 </robot>

File: ca_description/urdf/create_base.urdf.xacro (robot description, xacro)
@@ -28,5 +28,5 @@
     </joint>
   </xacro:macro>
-  <xacro:macro name="create_base" params="diffdrive_update_rate:=40 wheel_separation wheel_radius:=0.036 wheel_width:=0.024 wheel_torque:=1.0 wheel_accel:=1.8 mass_kg:=3.5 base_diameter *mesh">
+  <xacro:macro name="create_base" params="diffdrive_update_rate:=40 wheel_separation wheel_radius:=0.036 wheel_width:=0.024 wheel_torque:=1.0 wheel_accel:=1.8 mass_kg:=3.5 base_diameter *mesh visualize:=false">
     <xacro:include filename="$(find ca_description)/urdf/create_base_gazebo.urdf.xacro" />
     <link name="base_footprint">
@@ -172,6 +172,6 @@
     <!-- Simulation sensors -->
     <xacro:sim_create_base/>
-    <xacro:sim_create_wall_sensor/>
-    <xacro:sim_create_cliff_sensors/>
+    <xacro:sim_create_wall_sensor visualize="${visualize}"/>
+    <xacro:sim_create_cliff_sensors visualize="${visualize}"/>
     <xacro:sim_imu/>
   </xacro:macro>

File: ca_description/urdf/create_base_gazebo.urdf.xacro (robot description, xacro)
@@ -83,5 +83,5 @@
     </gazebo>
   </xacro:macro>
-  <xacro:macro name="sim_create_wall_sensor">
+  <xacro:macro name="sim_create_wall_sensor" params="visualize:=false">
     <gazebo reference="wall_sensor_link">
       <sensor type="ray" name="wall_sensor">
@@ -89,5 +89,5 @@
         <update_rate>20.0</update_rate>
         <pose>0 0 0 0 0 0</pose>
-        <visualize>false</visualize>
+        <visualize>${visualize}</visualize>
         <ray>
           <scan>
@@ -108,5 +108,5 @@
     </gazebo>
   </xacro:macro>
-  <xacro:macro name="sim_create_cliff_sensors">
+  <xacro:macro name="sim_create_cliff_sensors" params="visualize:=false">
     <gazebo reference="left_cliff_sensor_link">
       <sensor type="ray" name="left_cliff_sensor">
@@ -114,5 +114,5 @@
         <update_rate>20.0</update_rate>
         <pose>0 0 0 0 0 0</pose>
-        <visualize>false</visualize>
+        <visualize>${visualize}</visualize>
         <ray>
           <scan>
@@ -137,5 +137,5 @@
         <update_rate>20.0</update_rate>
         <pose>0 0 0 0 0 0</pose>
-        <visualize>false</visualize>
+        <visualize>${visualize}</visualize>
         <ray>
           <scan>
@@ -160,5 +160,5 @@
         <update_rate>20.0</update_rate>
         <pose>0 0 0 0 0 0</pose>
-        <visualize>false</visualize>
+        <visualize>${visualize}</visualize>
         <ray>
           <scan>
@@ -183,5 +183,5 @@
         <update_rate>20.0</update_rate>
         <pose>0 0 0 0 0 0</pose>
-        <visualize>false</visualize>
+        <visualize>${visualize}</visualize>
         <ray>
           <scan>

File: ca_description/urdf/roomblock.urdf.xacro (robot description, xacro)
@@ -12,5 +12,5 @@
     <color rgba="0.2 0.2 0.2 1.0"/>
   </material>
-  <xacro:macro name="roomblock">
+  <xacro:macro name="roomblock" params="visualize:=false">
     <joint name="block_joint" type="fixed">
       <origin xyz="0 0 ${block_z_offset}" rpy="0 0 0" />
@@ -40,5 +40,5 @@
     <link name="raspicam_link"/>
     <!-- Gazebo properties -->
-    <xacro:roomblock_gazebo/>
+    <xacro:roomblock_gazebo visualize="$(arg visualize)"/>
   </xacro:macro>
 </robot>

File: ca_description/urdf/roomblock_gazebo.urdf.xacro (robot description, xacro)
@@ -1,5 +1,5 @@
 <?xml version="1.0" ?>
 <robot xmlns:xacro="http://ros.org/wiki/xacro">
-  <xacro:macro name="roomblock_gazebo">
+  <xacro:macro name="roomblock_gazebo" params="visualize:=false">
     <gazebo reference="block_link">
       <material>Gazebo/Grey</material>
@@ -9,5 +9,5 @@
       <sensor type="ray" name="rplidar_sensor">
         <pose>0 0 0 0 0 0</pose>
-        <visualize>false</visualize>
+        <visualize>${visualize}</visualize>
         <update_rate>40</update_rate>
         <ray>
