Commit message: Modify wheel velocities and accelerations of the wheels

File: ca_description/urdf/create_base.urdf.xacro (robot description, xacro)
@@ -28,5 +28,5 @@
     </joint>
   </xacro:macro>
-  <xacro:macro name="create_base" params="diffdrive_update_rate:=40 wheel_separation wheel_radius:=0.036 wheel_width:=0.024 wheel_torque:=1.0 wheel_accel:=1.8 mass_kg:=3.5 base_diameter *mesh visualize:=false">
+  <xacro:macro name="create_base" params="diffdrive_update_rate:=40 wheel_separation wheel_radius:=0.036 wheel_width:=0.024 wheel_torque:=0.5 wheel_accel:=0.5 mass_kg:=3.5 base_diameter *mesh visualize:=false">
     <xacro:include filename="$(find ca_description)/urdf/create_base_gazebo.urdf.xacro" />
     <link name="base_footprint">

Commit message: Cleanup XACRO files

File: ca_description/urdf/create_base.urdf.xacro (robot description, xacro)
@@ -1,33 +1,11 @@
 <?xml version="1.0" ?>
 <robot xmlns:xacro="http://ros.org/wiki/xacro">
-  <xacro:macro name="create_wheel" params="prefix y_offset wheel_radius wheel_width">
-    <link name="${prefix}_wheel_link">
-    <inertial>
-      <origin xyz="0 0 0" />
-      <mass value="0.01" />
-      <inertia ixx="0.001" ixy="0.0" ixz="0.0" iyy="0.001" iyz="0.0" izz="0.001" />
-    </inertial>
-    <visual>
-      <origin xyz="0 0 0" rpy="0 ${pi/2} ${pi/2}" />
-      <geometry>
-        <cylinder radius="${wheel_radius}" length="${wheel_width}" />
-      </geometry>
-    </visual>
-    <collision>
-      <origin xyz="0 0 0" rpy="0 ${pi/2} ${pi/2}" />
-      <geometry>
-        <cylinder radius="${wheel_radius}" length="${wheel_width}" />
-      </geometry>
-    </collision>
-    </link>
-   <joint name="${prefix}_wheel_joint" type="continuous">
-      <origin xyz="0 ${y_offset} 0.015" rpy="0 0 0" />
-      <parent link="base_link" />
-      <child link="${prefix}_wheel_link" />
-      <axis xyz="0 1 0" />
-    </joint>
-  </xacro:macro>
   <xacro:macro name="create_base" params="diffdrive_update_rate:=40 wheel_separation wheel_radius:=0.036 wheel_width:=0.024 wheel_torque:=0.5 wheel_accel:=0.5 mass_kg:=3.5 base_diameter *mesh visualize:=false">
-    <xacro:include filename="$(find ca_description)/urdf/create_base_gazebo.urdf.xacro" />
+    <xacro:include filename="$(find ca_description)/urdf/create_base_gazebo.urdf.xacro"/>
+    <xacro:include filename="$(find ca_description)/urdf/create_caster_wheel.xacro"/>
+    <xacro:include filename="$(find ca_description)/urdf/create_wheel.xacro"/>
+    <xacro:include filename="$(find ca_description)/urdf/sensors/imu_sensor.xacro"/>
+    <xacro:include filename="$(find ca_description)/urdf/sensors/wall_sensor.xacro"/>
+    <xacro:include filename="$(find ca_description)/urdf/sensors/cliff_sensors.xacro"/>
     <link name="base_footprint">
     <visual>
@@ -46,56 +24,21 @@
     </link>
     <link name="base_link">
-    <inertial>
-      <mass value="2" />
-      <origin xyz="0 0 0.0" />
-      <inertia ixx="0.01" ixy="0.0" ixz="0.0" iyy="0.01" iyz="0.0" izz="0.5" />
-    </inertial>
-    <visual>
-      <origin xyz=" 0 0 0.0308" rpy="0 0 0" />
-      <geometry>
-        <xacro:insert_block name="mesh" />
-      </geometry>
-    </visual>
-    <collision>
-      <origin xyz="0.0 0.0 0.0308" rpy="0 0 0" />
-      <geometry>
-        <cylinder length="0.0611632" radius="0.16495" />
-      </geometry>
-    </collision>
-    </link>
-    <link name="wall_sensor_link">
-    <inertial>
-      <mass value="0.01" />
-      <origin xyz="0 0 0" />
-      <inertia ixx="0.001" ixy="0.0" ixz="0.0" iyy="0.001" iyz="0.0" izz="0.001" />
-    </inertial>
-    </link>
-    <link name="left_cliff_sensor_link">
-    <inertial>
-      <mass value="0.01" />
-      <origin xyz="0 0 0" />
-      <inertia ixx="0.001" ixy="0.0" ixz="0.0" iyy="0.001" iyz="0.0" izz="0.001" />
-    </inertial>
-    </link>
-    <link name="right_cliff_sensor_link">
-    <inertial>
-      <mass value="0.01" />
-      <origin xyz="0 0 0" />
-      <inertia ixx="0.001" ixy="0.0" ixz="0.0" iyy="0.001" iyz="0.0" izz="0.001" />
-    </inertial>
-    </link>
-    <link name="leftfront_cliff_sensor_link">
-    <inertial>
-      <mass value="0.01" />
-      <origin xyz="0 0 0" />
-      <inertia ixx="1.0" ixy="0.0" ixz="0.0" iyy="0.01" iyz="0.0" izz="0.01" />
-    </inertial>
-    </link>
-    <link name="rightfront_cliff_sensor_link">
-    <inertial>
-      <mass value="0.01" />
-      <origin xyz="0 0 0" />
-      <inertia ixx="0.001" ixy="0.0" ixz="0.0" iyy="0.001" iyz="0.0" izz="0.001" />
-    </inertial>
+      <inertial>
+        <mass value="2" />
+        <origin xyz="0 0 0.0" />
+        <inertia ixx="0.01" ixy="0.0" ixz="0.0" iyy="0.01" iyz="0.0" izz="0.5" />
+      </inertial>
+      <visual>
+        <origin xyz=" 0 0 0.0308" rpy="0 0 0" />
+        <geometry>
+          <xacro:insert_block name="mesh" />
+        </geometry>
+      </visual>
+      <collision>
+        <origin xyz="0.0 0.0 0.0308" rpy="0 0 0" />
+        <geometry>
+          <cylinder length="0.0611632" radius="0.16495" />
+        </geometry>
+      </collision>
     </link>
     <joint name="base_footprint_joint" type="fixed">
@@ -104,75 +47,12 @@
       <child link="base_link" />
     </joint>
-    <joint name="base_wall_sensor_joint" type="fixed">
-      <origin xyz="0.09 -0.120 0.042" rpy="0 0 -1.0" />
-      <parent link="base_link" />
-      <child link="wall_sensor_link" />
-    </joint>
-    <joint name="base_left_cliff_sensor_joint" type="fixed">
-      <origin xyz="0.07 0.14 0.01" rpy="0 ${pi/2} 0" />
-      <parent link="base_link" />
-      <child link="left_cliff_sensor_link" />
-    </joint>
-    <joint name="base_right_cliff_sensor_joint" type="fixed">
-      <origin xyz="0.07 -0.14 0.01" rpy="0 ${pi/2} 0" />
-      <parent link="base_link" />
-      <child link="right_cliff_sensor_link" />
-    </joint>
-    <joint name="base_leftfront_cliff_sensor_joint" type="fixed">
-      <origin xyz="0.15 0.04 0.01" rpy="0 ${pi/2} 0" />
-      <parent link="base_link" />
-      <child link="leftfront_cliff_sensor_link" />
-    </joint>
-    <joint name="base_rightfront_cliff_sensor_joint" type="fixed">
-      <origin xyz="0.15 -0.04 0.01" rpy="0 ${pi/2} 0" />
-      <parent link="base_link" />
-      <child link="rightfront_cliff_sensor_link" />
-    </joint>
+    <xacro:wall_sensor visualize="${visualize}"/>
+    <xacro:cliff_sensors visualize="${visualize}"/>
+    <xacro:imu_sensor/>
     <xacro:create_wheel prefix="left" y_offset="${wheel_separation / 2}" wheel_radius="${wheel_radius}" wheel_width="${wheel_width}"/>
     <xacro:create_wheel prefix="right" y_offset="${wheel_separation / -2}" wheel_radius="${wheel_radius}" wheel_width="${wheel_width}"/>
-    <link name="front_wheel_link">
-    <inertial>
-      <origin xyz="0 0 0" />
-      <mass value="0.01" />
-      <inertia ixx="0.001" ixy="0.0" ixz="0.0" iyy="0.001" iyz="0.0" izz="0.001" />
-    </inertial>
-    <visual>
-      <origin xyz="0 0 0" rpy="0 ${pi/2} ${pi/2}" />
-      <geometry>
-        <sphere radius="0.018" />
-      </geometry>
-    </visual>
-    <collision>
-      <origin xyz="0 0 0" rpy="0 ${pi/2} ${pi/2}" />
-      <geometry>
-        <sphere radius="0.018" />
-      </geometry>
-    </collision>
-    </link>
-    <!-- fixed because there's no transmission -->
-    <joint name="front_castor_joint" type="fixed">
-      <origin xyz="0.13 0 0.0" rpy="0 0 0" />
-      <parent link="base_link" />
-      <child link="front_wheel_link" />
-      <axis xyz="0 1 0" />
-    </joint>
-    <joint name="gyro_joint" type="fixed">
-      <axis xyz="0 1 0" />
-      <origin xyz="0 0 0.04" rpy="0 0 0" />
-      <parent link="base_link" />
-      <child link="gyro_link" />
-    </joint>
-    <link name="gyro_link">
-    <inertial>
-      <mass value="0.001" />
-      <origin xyz="0 0 0" rpy="0 0 0" />
-      <inertia ixx="0.0001" ixy="0" ixz="0" iyy="0.000001" iyz="0" izz="0.0001" />
-    </inertial>
-    </link>
+    <xacro:caster_wheel/>
     <!-- Simulation sensors -->
     <xacro:sim_create_base/>
-    <xacro:sim_create_wall_sensor visualize="${visualize}"/>
-    <xacro:sim_create_cliff_sensors visualize="${visualize}"/>
-    <xacro:sim_imu/>
   </xacro:macro>
 </robot>

File: ca_description/urdf/create_base_gazebo.urdf.xacro (robot description, xacro)
@@ -69,156 +69,3 @@
     </gazebo>
   </xacro:macro>
-  <xacro:macro name="sim_imu">
-    <gazebo>
-      <plugin name="imu_controller" filename="libgazebo_ros_imu.so">
-        <alwaysOn>true</alwaysOn>
-        <updateRate>30</updateRate>
-        <bodyName>gyro_link</bodyName>
-        <topicName>imu/data</topicName>
-        <serviceName>imu/is_calibrated</serviceName>
-        <gaussianNoise>${0.0017*0.0017}</gaussianNoise>
-        <xyzOffsets>0 0 0</xyzOffsets>
-        <rpyOffsets>0 0 0</rpyOffsets>
-      </plugin>
-    </gazebo>
-  </xacro:macro>
-  <xacro:macro name="sim_create_wall_sensor" params="visualize:=false">
-    <gazebo reference="wall_sensor_link">
-      <sensor type="ray" name="wall_sensor">
-        <always_on>true</always_on>
-        <update_rate>20.0</update_rate>
-        <pose>0 0 0 0 0 0</pose>
-        <visualize>${visualize}</visualize>
-        <ray>
-          <scan>
-            <horizontal>
-              <samples>1</samples>
-              <resolution>1</resolution>
-              <min_angle>0</min_angle>
-              <max_angle>0</max_angle>
-            </horizontal>
-          </scan>
-          <range>
-            <min>0.0160</min>
-            <max>0.04</max>
-            <resolution>0.1</resolution>
-          </range>
-        </ray>
-        <plugin name="gazebo_ros_wall_sensor" filename="libgazebo_ros_laser.so">
-          <topicName>/wall_sensor/scan</topicName>
-          <frameName>wall_sensor_link</frameName>
-        </plugin>
-      </sensor>
-    </gazebo>
-  </xacro:macro>
-  <xacro:macro name="sim_create_cliff_sensors" params="visualize:=false">
-    <gazebo reference="left_cliff_sensor_link">
-      <sensor type="ray" name="left_cliff_sensor">
-        <always_on>true</always_on>
-        <update_rate>20.0</update_rate>
-        <pose>0 0 0 0 0 0</pose>
-        <visualize>${visualize}</visualize>
-        <ray>
-          <scan>
-            <horizontal>
-              <samples>1</samples>
-              <resolution>1</resolution>
-              <min_angle>0</min_angle>
-              <max_angle>0</max_angle>
-            </horizontal>
-          </scan>
-          <range>
-            <min>0.01</min>
-            <max>0.04</max>
-            <resolution>0.1</resolution>
-          </range>
-        </ray>
-        <plugin name="gazebo_ros_left_side_cliff_sensor" filename="libgazebo_ros_laser.so">
-          <topicName>/left_side_cliff_sensor/scan</topicName>
-          <frameName>left_side_cliff_sensor_link</frameName>
-        </plugin>
-      </sensor>
-    </gazebo>
-    <gazebo reference="right_cliff_sensor_link">
-      <sensor type="ray" name="right_cliff_sensor">
-        <always_on>true</always_on>
-        <update_rate>20.0</update_rate>
-        <pose>0 0 0 0 0 0</pose>
-        <visualize>${visualize}</visualize>
-        <ray>
-          <scan>
-            <horizontal>
-              <samples>1</samples>
-              <resolution>1</resolution>
-              <min_angle>0</min_angle>
-              <max_angle>0</max_angle>
-            </horizontal>
-          </scan>
-          <range>
-            <min>0.01</min>
-            <max>0.04</max>
-            <resolution>0.1</resolution>
-          </range>
-        </ray>
-        <plugin name="gazebo_ros_right_side_cliff_sensor" filename="libgazebo_ros_laser.so">
-          <topicName>/right_side_cliff_sensor/scan</topicName>
-          <frameName>right_side_cliff_sensor_link</frameName>
-        </plugin>
-      </sensor>
-    </gazebo>
-    <gazebo reference="leftfront_cliff_sensor_link">
-      <sensor type="ray" name="leftfront_cliff_sensor">
-        <always_on>true</always_on>
-        <update_rate>20.0</update_rate>
-        <pose>0 0 0 0 0 0</pose>
-        <visualize>${visualize}</visualize>
-        <ray>
-          <scan>
-            <horizontal>
-              <samples>1</samples>
-              <resolution>1</resolution>
-              <min_angle>0</min_angle>
-              <max_angle>0</max_angle>
-            </horizontal>
-          </scan>
-          <range>
-            <min>0.01</min>
-            <max>0.04</max>
-            <resolution>0.1</resolution>
-          </range>
-        </ray>
-        <plugin name="gazebo_ros_left_front_cliff_sensor" filename="libgazebo_ros_laser.so">
-          <topicName>/left_front_cliff_sensor/scan</topicName>
-          <frameName>leftfront_cliff_sensor</frameName>
-        </plugin>
-      </sensor>
-    </gazebo>
-    <gazebo reference="rightfront_cliff_sensor_link">
-      <sensor type="ray" name="rightfront_cliff_sensor">
-        <always_on>true</always_on>
-        <update_rate>20.0</update_rate>
-        <pose>0 0 0 0 0 0</pose>
-        <visualize>${visualize}</visualize>
-        <ray>
-          <scan>
-            <horizontal>
-              <samples>1</samples>
-              <resolution>1</resolution>
-              <min_angle>0</min_angle>
-              <max_angle>0</max_angle>
-            </horizontal>
-          </scan>
-          <range>
-            <min>0.01</min>
-            <max>0.04</max>
-            <resolution>0.1</resolution>
-          </range>
-        </ray>
-        <plugin name="gazebo_ros_right_front_cliff_sensor" filename="libgazebo_ros_laser.so">
-          <topicName>/right_front_cliff_sensor/scan</topicName>
-          <frameName>rightfront_cliff_sensor</frameName>
-        </plugin>
-      </sensor>
-    </gazebo>
-  </xacro:macro>
 </robot>
