Commit message: feat: bumper sensor tested

File: create_description/urdf/create_1.urdf.xacro (robot description, xacro)
@@ -1,7 +1,8 @@
 <?xml version="1.0" ?>
-<robot name="create_1" xmlns:xacro="http://ros.org/wiki/xacro">
+<robot name="create_1"
+  xmlns:xacro="http://ros.org/wiki/xacro">
   <xacro:include filename="$(find create_description)/urdf/create_base.urdf.xacro" />
   <xacro:include filename="$(find create_description)/urdf/create_1_gazebo.urdf.xacro" />
-  <xacro:create_base wheel_separation="0.26" base_diameter="0.3302">
+  <xacro:create_base wheel_separation="0.26" base_diameter="0.3302" version="1">
     <mesh filename="package://create_description/meshes/create_1.dae" />
   </xacro:create_base>

File: create_description/urdf/create_2.urdf.xacro (robot description, xacro)
@@ -1,7 +1,8 @@
 <?xml version="1.0" ?>
-<robot name="create_2" xmlns:xacro="http://ros.org/wiki/xacro">
+<robot name="create_2"
+  xmlns:xacro="http://ros.org/wiki/xacro">
   <xacro:include filename="$(find create_description)/urdf/create_base.urdf.xacro" />
   <xacro:include filename="$(find create_description)/urdf/create_2_gazebo.urdf.xacro" />
-  <xacro:create_base wheel_separation="0.235" base_diameter="0.3485">
+  <xacro:create_base wheel_separation="0.235" base_diameter="0.3485" version="2">
     <mesh filename="package://create_description/meshes/create_2.dae" />
   </xacro:create_base>

File: create_description/urdf/create_base.urdf.xacro (robot description, xacro)
@@ -29,5 +29,5 @@
     </joint>
   </xacro:macro>
-  <xacro:macro name="create_base" params="diffdrive_update_rate:=40 wheel_separation wheel_radius:=0.036 wheel_width:=0.024 wheel_torque:=1.0 wheel_accel:=1.8 mass_kg:=3.5 base_diameter *mesh">
+  <xacro:macro name="create_base" params="diffdrive_update_rate:=40 wheel_separation wheel_radius:=0.036 wheel_width:=0.024 wheel_torque:=1.0 wheel_accel:=1.8 mass_kg:=3.5 base_diameter version *mesh">
     <xacro:include filename="$(find create_description)/urdf/create_base_gazebo.urdf.xacro" />
     <link name="base_footprint">
@@ -137,16 +137,10 @@
         <origin xyz="0 0 0" rpy="0 0 0"/>
         <geometry>
-          <box size="0.1 0.001 0.001"/>
-        </geometry>
-      </collision>
-      <visual>
-        <origin xyz="0 0 0" rpy="0 0 0"/>
-        <geometry>
-          <box size="0.1 0.001 0.001"/>
-        </geometry>
-      </visual>
+          <mesh filename="package://create_description/meshes/bumper_${version}.dae"/>
+        </geometry>
+      </collision>
     </link>
     <joint name="bumper_joint" type="fixed">
-      <origin xyz="${base_diameter/2} 0 0" rpy="0 0 0" />
+      <origin xyz="-0.0025 0 0" rpy="0 0 0" />
       <parent link="base_link" />
       <child link="bumper_link" />
@@ -232,5 +226,5 @@
     <xacro:sim_imu/>
     <xacro:sim_bumper/>
-    <xacro:sim_ir/>
+    <!-- <xacro:sim_ir/> -->
   </xacro:macro>
 </robot>

File: create_description/urdf/create_base_gazebo.urdf.xacro (robot description, xacro)
@@ -81,5 +81,5 @@
       <sensor name="sim_bumper" type="contact">
         <alwaysOn>true</alwaysOn>
-        <updateRate>20.0</updateRate>
+        <updateRate>1000.0</updateRate>
         <material>Gazebo/Red</material>
         <contact>
