Commit message: feat: minimal sensor config

File: create_description/urdf/create_base.urdf.xacro (robot description, xacro)
@@ -4,23 +4,23 @@
   <xacro:macro name="create_wheel" params="prefix y_offset wheel_radius wheel_width">
     <link name="${prefix}_wheel_link">
-    <inertial>
-      <origin xyz="0 0 0" />
-      <mass value="0.01" />
-      <inertia ixx="0.001" ixy="0.0" ixz="0.0" iyy="0.001" iyz="0.0" izz="0.001" />
-    </inertial>
-    <visual>
-      <origin xyz="0 0 0" rpy="0 ${PI/2} ${PI/2}" />
-      <geometry>
-        <cylinder radius="${wheel_radius}" length="${wheel_width}" />
-      </geometry>
-    </visual>
-    <collision>
-      <origin xyz="0 0 0" rpy="0 ${PI/2} ${PI/2}" />
-      <geometry>
-        <cylinder radius="${wheel_radius}" length="${wheel_width}" />
-      </geometry>
-    </collision>
-    </link>
-   <joint name="${prefix}_wheel_joint" type="continuous">
+      <inertial>
+        <origin xyz="0 0 0" />
+        <mass value="0.01" />
+        <inertia ixx="0.001" ixy="0.0" ixz="0.0" iyy="0.001" iyz="0.0" izz="0.001" />
+      </inertial>
+      <visual>
+        <origin xyz="0 0 0" rpy="0 ${PI/2} ${PI/2}" />
+        <geometry>
+          <cylinder radius="${wheel_radius}" length="${wheel_width}" />
+        </geometry>
+      </visual>
+      <collision>
+        <origin xyz="0 0 0" rpy="0 ${PI/2} ${PI/2}" />
+        <geometry>
+          <cylinder radius="${wheel_radius}" length="${wheel_width}" />
+        </geometry>
+      </collision>
+    </link>
+    <joint name="${prefix}_wheel_joint" type="continuous">
       <origin xyz="0 ${y_offset} 0.015" rpy="0 0 0" />
       <parent link="base_link" />
@@ -32,71 +32,71 @@
     <xacro:include filename="$(find create_description)/urdf/create_base_gazebo.urdf.xacro" />
     <link name="base_footprint">
-    <visual>
-      <origin xyz="0 0 0" rpy="0 0 0" />
-      <geometry>
-        <box size="0.001 0.001 0.001" />
-      </geometry>
-      <material name="Green" />
-    </visual>
-    <collision>
-      <origin xyz="0 0 0.017" rpy="0 0 0" />
-      <geometry>
-        <box size="0.001 0.001 0.001" />
-      </geometry>
-    </collision>
+      <visual>
+        <origin xyz="0 0 0" rpy="0 0 0" />
+        <geometry>
+          <box size="0.001 0.001 0.001" />
+        </geometry>
+        <material name="Green" />
+      </visual>
+      <collision>
+        <origin xyz="0 0 0.017" rpy="0 0 0" />
+        <geometry>
+          <box size="0.001 0.001 0.001" />
+        </geometry>
+      </collision>
     </link>
     <link name="base_link">
-    <inertial>
-      <mass value="2" />
-      <origin xyz="0 0 0.0" />
-      <inertia ixx="0.01" ixy="0.0" ixz="0.0" iyy="0.01" iyz="0.0" izz="0.5" />
-    </inertial>
-    <visual>
-      <origin xyz=" 0 0 0.0308" rpy="0 0 0" />
-      <geometry>
-        <xacro:insert_block name="mesh" />
-      </geometry>
-    </visual>
-    <collision>
-      <origin xyz="0.0 0.0 0.0308" rpy="0 0 0" />
-      <geometry>
-        <cylinder length="0.0611632" radius="0.16495" />
-      </geometry>
-    </collision>
+      <inertial>
+        <mass value="2" />
+        <origin xyz="0 0 0.0" />
+        <inertia ixx="0.01" ixy="0.0" ixz="0.0" iyy="0.01" iyz="0.0" izz="0.5" />
+      </inertial>
+      <visual>
+        <origin xyz=" 0 0 0.0308" rpy="0 0 0" />
+        <geometry>
+          <xacro:insert_block name="mesh" />
+        </geometry>
+      </visual>
+      <collision>
+        <origin xyz="0.0 0.0 0.0308" rpy="0 0 0" />
+        <geometry>
+          <cylinder length="0.0611632" radius="0.16495" />
+        </geometry>
+      </collision>
     </link>
     <link name="wall_sensor_link">
-    <inertial>
-      <mass value="0.01" />
-      <origin xyz="0 0 0" />
-      <inertia ixx="0.001" ixy="0.0" ixz="0.0" iyy="0.001" iyz="0.0" izz="0.001" />
-    </inertial>
+      <inertial>
+        <mass value="0.01" />
+        <origin xyz="0 0 0" />
+        <inertia ixx="0.001" ixy="0.0" ixz="0.0" iyy="0.001" iyz="0.0" izz="0.001" />
+      </inertial>
     </link>
     <link name="left_cliff_sensor_link">
-    <inertial>
-      <mass value="0.01" />
-      <origin xyz="0 0 0" />
-      <inertia ixx="0.001" ixy="0.0" ixz="0.0" iyy="0.001" iyz="0.0" izz="0.001" />
-    </inertial>
+      <inertial>
+        <mass value="0.01" />
+        <origin xyz="0 0 0" />
+        <inertia ixx="0.001" ixy="0.0" ixz="0.0" iyy="0.001" iyz="0.0" izz="0.001" />
+      </inertial>
     </link>
     <link name="right_cliff_sensor_link">
-    <inertial>
-      <mass value="0.01" />
-      <origin xyz="0 0 0" />
-      <inertia ixx="0.001" ixy="0.0" ixz="0.0" iyy="0.001" iyz="0.0" izz="0.001" />
-    </inertial>
+      <inertial>
+        <mass value="0.01" />
+        <origin xyz="0 0 0" />
+        <inertia ixx="0.001" ixy="0.0" ixz="0.0" iyy="0.001" iyz="0.0" izz="0.001" />
+      </inertial>
     </link>
     <link name="leftfront_cliff_sensor_link">
-    <inertial>
-      <mass value="0.01" />
-      <origin xyz="0 0 0" />
-      <inertia ixx="1.0" ixy="0.0" ixz="0.0" iyy="0.01" iyz="0.0" izz="0.01" />
-    </inertial>
+      <inertial>
+        <mass value="0.01" />
+        <origin xyz="0 0 0" />
+        <inertia ixx="1.0" ixy="0.0" ixz="0.0" iyy="0.01" iyz="0.0" izz="0.01" />
+      </inertial>
     </link>
     <link name="rightfront_cliff_sensor_link">
-    <inertial>
-      <mass value="0.01" />
-      <origin xyz="0 0 0" />
-      <inertia ixx="0.001" ixy="0.0" ixz="0.0" iyy="0.001" iyz="0.0" izz="0.001" />
-    </inertial>
+      <inertial>
+        <mass value="0.01" />
+        <origin xyz="0 0 0" />
+        <inertia ixx="0.001" ixy="0.0" ixz="0.0" iyy="0.001" iyz="0.0" izz="0.001" />
+      </inertial>
     </link>
     <joint name="base_footprint_joint" type="fixed">
@@ -132,10 +132,39 @@
     <xacro:create_wheel prefix="left" y_offset="${wheel_separation / 2}" wheel_radius="${wheel_radius}" wheel_width="${wheel_width}"/>
     <xacro:create_wheel prefix="right" y_offset="${wheel_separation / -2}" wheel_radius="${wheel_radius}" wheel_width="${wheel_width}"/>
+    <!-- bumper sensor link -->
+    <link name="bumper_link">
+      <collision name="bumper_link_collision">
+        <origin xyz="0 0 0" rpy="0 0 0"/>
+        <geometry>
+          <box size="0.1 0.001 0.001"/>
+        </geometry>
+      </collision>
+      <visual>
+        <origin xyz="0 0 0" rpy="0 0 0"/>
+        <geometry>
+          <box size="0.1 0.001 0.001"/>
+        </geometry>
+      </visual>
+    </link>
+    <joint name="bumper_joint" type="fixed">
+      <origin xyz="${base_diameter/2} 0 0" rpy="0 0 0" />
+      <parent link="base_link" />
+      <child link="bumper_link" />
+      <axis xyz="0 0 0" />
+    </joint>
+    <!-- omni_ir sensor link -->
+    <link name="omni_ir_link">
+    </link>
+    <joint name="omni_ir_joint" type="fixed">
+      <origin xyz="${base_diameter/2 - 0.025} 0 0.0775" rpy="0 0 0" />
+      <parent link="base_link" />
+      <child link="omni_ir_link" />
+      <axis xyz="0 0 0" />
+    </joint>
     <!--<link name="rear_wheel_link">
     <inertial>
       <origin xyz="0 0 0"/>
       <mass value="0.001" />
-      <inertia ixx="0.0001" ixy="0.0" ixz="0.0"
-        iyy="0.0001" iyz="0.0" izz="0.0001" />
+      <inertia ixx="0.0001" ixy="0.0" ixz="0.0" iyy="0.0001" iyz="0.0" izz="0.0001" />
     </inertial>
     <visual>
@@ -159,21 +188,21 @@
     </joint>-->
     <link name="front_wheel_link">
-    <inertial>
-      <origin xyz="0 0 0" />
-      <mass value="0.01" />
-      <inertia ixx="0.001" ixy="0.0" ixz="0.0" iyy="0.001" iyz="0.0" izz="0.001" />
-    </inertial>
-    <visual>
-      <origin xyz="0 0 0" rpy="0 ${PI/2} ${PI/2}" />
-      <geometry>
-        <sphere radius="0.018" />
-      </geometry>
-    </visual>
-    <collision>
-      <origin xyz="0 0 0" rpy="0 ${PI/2} ${PI/2}" />
-      <geometry>
-        <sphere radius="0.018" />
-      </geometry>
-    </collision>
+      <inertial>
+        <origin xyz="0 0 0" />
+        <mass value="0.01" />
+        <inertia ixx="0.001" ixy="0.0" ixz="0.0" iyy="0.001" iyz="0.0" izz="0.001" />
+      </inertial>
+      <visual>
+        <origin xyz="0 0 0" rpy="0 ${PI/2} ${PI/2}" />
+        <geometry>
+          <sphere radius="0.018" />
+        </geometry>
+      </visual>
+      <collision>
+        <origin xyz="0 0 0" rpy="0 ${PI/2} ${PI/2}" />
+        <geometry>
+          <sphere radius="0.018" />
+        </geometry>
+      </collision>
     </link>
     <!-- fixed because there's no transmission -->
@@ -191,9 +220,9 @@
     </joint>
     <link name="gyro_link">
-    <inertial>
-      <mass value="0.001" />
-      <origin xyz="0 0 0" rpy="0 0 0" />
-      <inertia ixx="0.0001" ixy="0" ixz="0" iyy="0.000001" iyz="0" izz="0.0001" />
-    </inertial>
+      <inertial>
+        <mass value="0.001" />
+        <origin xyz="0 0 0" rpy="0 0 0" />
+        <inertia ixx="0.0001" ixy="0" ixz="0" iyy="0.000001" iyz="0" izz="0.0001" />
+      </inertial>
     </link>
     <!-- Simulation sensors -->
@@ -202,4 +231,6 @@
     <xacro:sim_create_cliff_sensors/>
     <xacro:sim_imu/>
+    <xacro:sim_bumper/>
+    <xacro:sim_ir/>
   </xacro:macro>
 </robot>

File: create_description/urdf/create_base_gazebo.urdf.xacro (robot description, xacro)
@@ -77,4 +77,59 @@
     </gazebo>
   </xacro:macro>
+  <xacro:macro name="sim_bumper">
+    <gazebo reference="bumper_link">
+      <sensor name="sim_bumper" type="contact">
+        <alwaysOn>true</alwaysOn>
+        <updateRate>20.0</updateRate>
+        <material>Gazebo/Red</material>
+        <contact>
+          <collision>base_footprint_fixed_joint_lump__bumper_link_collision_collision_2</collision>
+        </contact>
+        <plugin name="gazebo_ros_bumper_controller" filename="libgazebo_ros_bumper.so">
+          <bumperTopicName>bumper</bumperTopicName>
+          <frameName>bumper_link</frameName>
+        </plugin>
+      </sensor>
+    </gazebo>
+  </xacro:macro>
+  <xacro:macro name="sim_ir">
+    <gazebo reference="omni_ir_link">
+      <sensor type="ray" name="TeraRanger">
+        <pose>0 0 0 0 0 0</pose>
+        <visualize>true</visualize>
+        <update_rate>50</update_rate>
+        <ray>
+          <scan>
+            <horizontal>
+              <samples>10</samples>
+              <resolution>1</resolution>
+              <min_angle>${-6.28319/2}</min_angle>
+              <max_angle>${6.28319/2}</max_angle>
+            </horizontal>
+            <vertical>
+              <samples>10</samples>
+              <resolution>1</resolution>
+              <min_angle>-0.14835</min_angle>
+              <max_angle>0.14835</max_angle>
+            </vertical>
+          </scan>
+          <range>
+            <min>0.01</min>
+            <max>2</max>
+            <resolution>0.02</resolution>
+          </range>
+        </ray>
+        <plugin filename="libgazebo_ros_range.so" name="gazebo_ros_range">
+          <gaussianNoise>0.005</gaussianNoise>
+          <alwaysOn>true</alwaysOn>
+          <updateRate>50</updateRate>
+          <topicName>omni_ir</topicName>
+          <frameName>omni_ir_link</frameName>
+          <radiation>INFRARED</radiation>
+          <fov>6.28319</fov>
+        </plugin>
+      </sensor>
+    </gazebo>
+  </xacro:macro>
   <xacro:macro name="sim_create_wall_sensor">
     <gazebo reference="wall_sensor_link">

Commit message: chore: erasing changes

File: create_description/urdf/create_base.urdf.xacro (robot description, xacro)
@@ -226,5 +226,4 @@
     <xacro:sim_imu/>
     <xacro:sim_bumper/>
-    <xacro:sim_ir/>
   </xacro:macro>
 </robot>

File: create_description/urdf/create_base_gazebo.urdf.xacro (robot description, xacro)
@@ -93,43 +93,4 @@
     </gazebo>
   </xacro:macro>
-  <xacro:macro name="sim_ir">
-    <gazebo reference="omni_ir_link">
-      <sensor type="ray" name="TeraRanger">
-        <pose>0 0 0 0 0 0</pose>
-        <visualize>true</visualize>
-        <update_rate>50</update_rate>
-        <ray>
-          <scan>
-            <horizontal>
-              <samples>10</samples>
-              <resolution>1</resolution>
-              <min_angle>${-0.14835*2}</min_angle>
-              <max_angle>${0.14835*2}</max_angle>
-            </horizontal>
-            <vertical>
-              <samples>10</samples>
-              <resolution>1</resolution>
-              <min_angle>-0.05</min_angle>
-              <max_angle>0.05</max_angle>
-            </vertical>
-          </scan>
-          <range>
-            <min>0.01</min>
-            <max>2</max>
-            <resolution>0.02</resolution>
-          </range>
-        </ray>
-        <plugin filename="libgazebo_ros_range.so" name="gazebo_ros_range">
-          <gaussianNoise>0.005</gaussianNoise>
-          <alwaysOn>true</alwaysOn>
-          <updateRate>50</updateRate>
-          <topicName>omni_ir</topicName>
-          <frameName>omni_ir_link</frameName>
-          <radiation>INFRARED</radiation>
-          <fov>${0.14835*2}</fov>
-        </plugin>
-      </sensor>
-    </gazebo>
-  </xacro:macro>
   <xacro:macro name="sim_create_wall_sensor">
     <gazebo reference="wall_sensor_link">
